File: Hardware/sbs2-board/sbs2-board.kicad_pcb (KiCad board)
At the start: 2 copper layers, 100 x 70 mm, 83 parts, among them J401 Conn_01x14_Male, J402 Conn_01x14_Male, J403 Conn_01x07_Male, J404 Conn_01x06_Male, J406 Conn_02x03_Counter_Clockwise, J407 Conn_02x03_Counter_Clockwise, Q201 SS8050, Q202 SS8050, Q301 PW2320, Q302 PW8205A8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

Commit message: 更新电路图
Parts:
- removed C3012: 22uF, Capacitor_SMD:C_0805_2012Metric
- removed H5, H6, H7, H8: MountingHole, MountingHole:MountingHole_2.2mm_M2_ISO14580
- added C312: 22uF, Capacitor_SMD:C_0805_2012Metric, F.Cu at (148.5, 76.0)
- added C314: 22pF, Capacitor_SMD:C_0805_2012Metric, F.Cu at (137.0, 71.0)
- J406, J407: value Conn_02x03_Counter_Clockwise -> Conn_02x03_Odd_Even
- moved C301 298.0 mm to (120.0, 106.0)
- moved R301 297.4 mm to (124.0, 106.0)
- moved R308 294.3 mm to (139.0, 71.0), turned to 90 degrees
- moved C305 294.1 mm to (153.0, 109.0), turned to -90 degrees
- moved R304 291.4 mm to (171.5, 117.0), turned to -90 degrees
- moved C303 289.1 mm to (120.0, 110.0), turned to 180 degrees
- moved C302 288.4 mm to (120.0, 108.0)
- moved R309 288.3 mm to (135.0, 75.5), turned to 90 degrees
- moved J407 286.8 mm to (152.5, 75.0)
- moved R306 286.6 mm to (160.0, 109.0), turned to 90 degrees
- moved C304 285.5 mm to (155.0, 109.0), turned to -90 degrees
- moved U301 281.6 mm to (137.0, 105.0), turned to 180 degrees
- moved D303 281.3 mm to (134.0, 91.0), turned to 180 degrees
- moved D301 280.1 mm to (149.0, 114.0), turned to 180 degrees
- moved J406 278.4 mm to (152.5, 65.0)
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Connections:
- net Net-(C310-Pad2) renamed /LC301
- net Net-(D301-Pad2) renamed /LD301
- net Net-(L301-Pad1) renamed /LR301
- net Net-(Q302-Pad1) renamed /DD301
- C101 pad 1: GND -> +5V
- C101 pad 2: +5V -> GND
- C102 pad 1: GND -> +5V
- C102 pad 2: +5V -> GND
- C313 pad 1: GND -> +3V3
- C313 pad 2: +3V3 -> GND
- J406 pad 2: +3V3 -> GND
- J406 pad 5: GND -> +3V3
- J407 pad 2: +3V3 -> GND
- J407 pad 5: GND -> +3V3
- Q303 pad 3: /BG -> Net-(SW301-Pad2)
- R310 pad 1: /BG -> Net-(SW301-Pad1)
- SW301 pad 1: unconnected-(SW301-Pad1) -> Net-(SW301-Pad1)
- SW301 pad 2: unconnected-(SW301-Pad2) -> Net-(SW301-Pad2)
- SW301 pad 3: unconnected-(SW301-Pad3) -> GND
- SW301 pad 4: /BG -> Net-(SW301-Pad1)
- SW301 pad 5: GND -> Net-(SW301-Pad2)
- SW301 pad 6: unconnected-(SW301-Pad6) -> GND
- U101 pad 13: +3V3 -> +5V
Routing:
- net +3V3: track 31.9 -> 273.2 mm, vias 0 -> 9
- net GND: track 194.4 -> 342.9 mm, vias 6 -> 44
- net /BAT: track 0.00 -> 133.0 mm, vias 0 -> 19
- net /ESP_TX: track 0.00 -> 90.3 mm, vias 0 -> 2
- net /ESP_RX: track 0.00 -> 89.3 mm, vias 0 -> 2
- net +5V: track 71.5 -> 154.6 mm, vias 10 -> 33
- net /ESP_IO0: track 59.3 -> 134.5 mm
- net Net-(BT1-Pad2): track 0.00 -> 63.8 mm, vias 0 -> 1
- net /BGND: track 0.00 -> 45.6 mm
- net Net-(Q302-Pad5): track 0.00 -> 30.5 mm, vias 0 -> 2
- net /ESP_EN: track 73.4 -> 102.4 mm
- net Net-(J402-Pad14): track 0.00 -> 21.1 mm
- net /BT-: track 0.00 -> 19.8 mm, vias 0 -> 6
- net Net-(Q302-Pad4): track 0.00 -> 19.8 mm, vias 0 -> 2
- net Net-(J402-Pad13): track 0.00 -> 17.9 mm
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- added copper zone on F.Cu, net +3V3
- added copper zone on F.Cu, net +5V
- added copper zone on F.Cu, net /BAT
- added copper zone on F.Cu, net /BGND
- added copper zone on F.Cu, net /BT-
- added copper zone on F.Cu, net /DD301
- added copper zone on F.Cu, net /LC301
- added copper zone on F.Cu, net /LD301
- added copper zone on F.Cu, net /LR301
- added copper zone on B.Cu, net GND
- added copper zone on F.Cu, net GND
- added copper zone on F.Cu, net VCC
Other:
- board text added: "13 12 11 10 09 08 07 06 05 04 03 02 01"
- board text added: "14 15 16 17 18 19 20"
- board text added: "21 26 33 34 35 36 37 38 39 40 41 42 45 46"
- board text added: "3 G V N 3 D"
- board text added: "BOOT"
- board text added: "EN"
- board text added: "IO0 EN GND RX TX 3V3"
- board text added: "JLCJLCJLCJLC"

Commit message: 更新电路图
Connections:
- C104 pad 1: +3V3 -> Net-(C104-Pad1)
- C105 pad 1: +3V3 -> Net-(C104-Pad1)
- J403 pad 3: /USB_2_D- -> Net-(J403-Pad3)
- J403 pad 4: /USB_2_D+ -> Net-(J403-Pad4)
- J403 pad 6: Net-(J403-Pad6) -> /USB_2_D-
- J403 pad 7: Net-(J403-Pad7) -> /USB_2_D+
- U101 pad 12: +3V3 -> Net-(C104-Pad1)
- U101 pad 14: unconnected-(U101-Pad14) -> Net-(C104-Pad1)
- U401 pad 19: /USB_2_D- -> Net-(J403-Pad3)
- U401 pad 20: /USB_2_D+ -> Net-(J403-Pad4)
- U401 pad 22: Net-(J403-Pad6) -> /USB_2_D-
- U401 pad 23: Net-(J403-Pad7) -> /USB_2_D+
Routing:
- net +3V3: track 273.2 -> 259.0 mm, vias 9 -> 8
- net Net-(J403-Pad7): track 11.3 -> 0.00 mm
- net Net-(J403-Pad6): track 10.9 -> 0.00 mm
- net Net-(J403-Pad3): track 0.00 -> 10.5 mm
- net Net-(J403-Pad4): track 0.00 -> 10.5 mm
- net /USB_2_D-: track 49.3 -> 59.4 mm
- net /USB_2_D+: track 50.8 -> 60.0 mm
- net Net-(C104-Pad1): track 0.00 -> 8.83 mm
