File: Hardware/sbs2-board/sbs2-board.kicad_sch (KiCad schematic)
At the start: 4 parts

Commit message: 更新电路图
Parts:
- added BT1, BT2: (no value), sb-board:BT-503450, symbol Device:Battery_Cell
- added C101, C102, C313: 100uF, Capacitor_SMD:CP_Elec_6.3x5.4, symbol Device:C_Small
- added C104, C201, C303, C306, C307, C309, C310, C311, C401: 100nF, Capacitor_SMD:C_0805_2012Metric, symbol Device:C_Small
- added C105, C202, C301, C402: 10uF, Capacitor_SMD:C_0805_2012Metric, symbol Device:C_Small
- added C3012, C302, C304, C305, C308: 22uF, Capacitor_SMD:C_0805_2012Metric, symbol Device:C_Small
- added C403: 1uF, Capacitor_SMD:C_0805_2012Metric, symbol Device:C_Small
- added D301, D302, D303: D1FH3, Diode_SMD:D_SMA, symbol Device:D
- added D401: LED_R, LED_SMD:LED_0603_1608Metric, symbol Device:LED_Small
- added D402: LED_B, LED_SMD:LED_0603_1608Metric, symbol Device:LED_Small
- added F101: 6V 1A, Fuse:Fuse_1206_3216Metric, symbol Device:Fuse_Small
- added H1, H2, H3, H4: MountingHole, MountingHole:MountingHole_3.2mm_M3_ISO14580, symbol Mechanical:MountingHole
- added H5, H6, H7, H8: MountingHole, MountingHole:MountingHole_2.2mm_M2_ISO14580, symbol Mechanical:MountingHole
- added J401, J402: Conn_01x14_Male, Connector_PinHeader_2.54mm:PinHeader_1x14_P2.54mm_Vertical, symbol Connector:Conn_01x14_Male
- added J403: Conn_01x07_Male, Connector_PinHeader_2.54mm:PinHeader_1x07_P2.54mm_Vertical, symbol Connector:Conn_01x07_Male
- added J404: Conn_01x06_Male, Connector_PinHeader_2.54mm:PinHeader_1x06_P2.54mm_Vertical, symbol Connector:Conn_01x06_Male
- added J406, J407: Conn_02x03_Counter_Clockwise, Connector_PinHeader_2.54mm:PinHeader_2x03_P2.54mm_Vertical, symbol Connector_Generic:Conn_02x03_Counter_Clockwise
- added L301: 10uH, Inductor_SMD:L_Abracon_ASPI-0630LR, symbol Device:L_Small
- added L302: 4.7uH, Inductor_SMD:L_Abracon_ASPI-0630LR, symbol Device:L_Small
- added Q201, Q202: SS8050, Package_TO_SOT_SMD:SOT-23, symbol Device:Q_NPN_BEC
- added Q301, Q303: PW2320, Package_TO_SOT_SMD:SOT-23, symbol Device:Q_NMOS_DSG
- added Q302: PW8205A8, Package_SO:TSSOP-8_4.4x3mm_P0.65mm, symbol sb-board:PW8205A8
- added R101: 5.1K, Resistor_SMD:R_0805_2012Metric, symbol Device:R_Small
- added R102, R307: 100K, Resistor_SMD:R_0805_2012Metric, symbol Device:R_Small
- added R201, R202, R310, R401, R402: 10K, Resistor_SMD:R_0805_2012Metric, symbol Device:R_Small
- added R301: 5R, Resistor_SMD:R_0805_2012Metric, symbol Device:R_Small
- added R302: 0.12R, Resistor_SMD:R_2512_6332Metric, symbol Device:R_Small
- added R303: 20R, Resistor_SMD:R_0805_2012Metric, symbol Device:R_Small
- added R304, R305: 330R, Resistor_SMD:R_0805_2012Metric, symbol Device:R_Small
- added R306: 1K, Resistor_SMD:R_0805_2012Metric, symbol Device:R_Small
- added R308: 47K, Resistor_SMD:R_0805_2012Metric, symbol Device:R_Small
- added R309: 15K, Resistor_SMD:R_0805_2012Metric, symbol Device:R_Small
- added R403, R404: 750, Resistor_SMD:R_0805_2012Metric, symbol Device:R_Small
- added SW301: SW_Push_DPDT, Button_Switch_THT:SW_E-Switch_EG1271_DPDT, symbol Switch:SW_Push_DPDT
- added SW401, SW402: SW_Push, Button_Switch_SMD:SW_SPST_CK_RS282G05A3, symbol Switch:SW_Push
- added U101: HS8836A, Package_SO:SOIC-16_3.9x9.9mm_P1.27mm, symbol sb-board:HS8836A
- added U201: CH340C, Package_SO:SOIC-16_3.9x9.9mm_P1.27mm, symbol Interface_USB:CH340C
- added U301: PW4202, Package_SO:SOIC-8_3.9x4.9mm_P1.27mm, symbol sb-board:PW4202
- added U302: PW7152, Package_TO_SOT_SMD:SOT-23-6, symbol sb-board:PW7152
- added U303: PW2312, Package_TO_SOT_SMD:SOT-23-6, symbol sb-board:PW2312
- added U401: ESP32-S2-WROVER, sb-board:ESP32-S2-WROVER-I, symbol sb-board:ESP32-S2-WROVER
- added U402: OLED_096_IIC, sb-board:OLED_096_IIC, symbol sb-board:OLED_096_IIC
- renumbered USB0101 to USB101, USB0102 to USB102, USB0103 to USB103, USB0104 to USB104
Connections:
- net GND: now also C101.1, C102.1, C104.2, C105.2, C201.1, C202.1, C3012.1, C308.1, C309.1, C311.1, C313.1, C401.2, C402.2, C403.1, D401.1 (K), D402.1 (K), J404.4 (Pin_4), J406.4 (Pin_4), J406.5 (Pin_5), J406.6 (Pin_6), J407.4 (Pin_4), J407.5 (Pin_5), J407.6 (Pin_6), Q303.2 (S), R101.2, R102.2, R309.1, SW301.5 (B), SW401.1, SW402.1, U101.16 (GND), U201.1 (GND), U303.2 (GND), U401.1 (GND), U401.26 (GND), U401.42 (GND), U401.43 (GND), U402.1 (Pin_1)
- net USB_IN_D+: now also U101.11 (DP)
- net USB_IN_D-: now also U101.10 (DM)
- net USB_IN_RX+: now also USB102.A11 (RX2+); no longer USB102.B11 (RX1+)
- net USB_IN_RX-: now also USB102.A10 (RX2-); no longer USB102.B10 (RX1-)
- net USB_IN_TX+: now also USB102.B2 (TX2+); no longer USB102.A2 (TX1+)
- net USB_IN_TX-: now also USB102.B3 (TX2-); no longer USB102.A3 (TX1-)
- net VIN: now also F101.1
- net +5V: now reaches USB103.1 (VBUS)
- net +5V: now also USB104.1 (VBUS), C101.2, C102.2, C302.2, C303.1, D302.2 (A), F101.2, R301.2, R302.2, U301.2 (CE), U301.7 (VIN)
- net USB_3_D-: now reaches USB103.2 (D-)
- net USB_3_D-: now also U101.3 (DM3)
- net USB_3_D+: now reaches USB103.3 (D+)
- net USB_3_D+: now also U101.4 (DP3)
- net at USB102.B5 (CC2): now also R101.1
- net USB_4_D-: now reaches USB104.2 (D-)
- net USB_4_D-: now also U101.1 (DM4)
- net USB_4_D+: now reaches USB104.3 (D+)
- net USB_4_D+: now also U101.2 (DP4)
- new net: J402.1 (Pin_1), U401.40 (IO46)
- new net: J402.10 (Pin_10), U401.29 (IO35)
- new net: J402.11 (Pin_11), U401.28 (IO34)
- new net: J402.12 (Pin_12), U401.27 (IO33)
- new net: J402.13 (Pin_13), U401.25 (IO26)
- new net: J402.14 (Pin_14), U401.24 (IO21)
- new net: J402.2 (Pin_2), U401.39 (IO45)
- new net: J402.3 (Pin_3), U401.36 (IO42)
- new net: J402.4 (Pin_4), U401.35 (IO41)
- new net: J402.5 (Pin_5), U401.34 (IO40)
- new net: J402.6 (Pin_6), U401.33 (IO39)
- new net: J402.7 (Pin_7), U401.32 (IO38)
- new net: J402.8 (Pin_8), U401.31 (IO37)
- new net: J402.9 (Pin_9), U401.30 (IO36)
- new net: BT1.2 (-), BT2.1 (+), R305.2
- new net: R303.2, U301.5 (LDRV)
- new net: L301.1, R302.1, U301.8 (CSN)
- new net: Q202.1 (B), R201.1
- new net: Q202.2 (E), R202.2, U201.14 (~{RTS})
- new net: Q201.1 (B), R202.1
- new net: Q201.2 (E), R201.2, U201.13 (~{DTR})
- new net: Q302.4 (G1), U302.1 (DOUT)
- new net: Q302.5 (G2), U302.2 (COUT)
- new net: R306.1, U302.3 (VM)
- new net: C307.2, R305.1, U302.4 (VC)
- new net: C306.2, R304.1, U302.5 (VDD)
- new net: D401.2 (A), R403.2
- new net: D301.2 (A), L301.2, Q301.1 (D)
- new net: J403.1 (Pin_1), U401.17 (IO14)
- new net: J403.2 (Pin_2), U401.18 (IO15)
- new net: J403.5 (Pin_5), U401.21 (IO18)
- new net: J403.6 (Pin_6), U401.22 (IO19)
- new net: J403.7 (Pin_7), U401.23 (IO20)
- new net: J401.8 (Pin_8), U401.10 (IO7)
- new net: J401.11 (Pin_11), U401.13 (IO10)
- new net: J401.12 (Pin_12), U401.14 (IO11)
- new net: J401.13 (Pin_13), U401.15 (IO12)
- new net: J401.14 (Pin_14), U401.16 (IO13)
- new net: J401.2 (Pin_2), U401.4 (IO1)
- new net: J401.4 (Pin_4), U401.6 (IO3)
- new net: J401.5 (Pin_5), U401.7 (IO4)
- new net: J401.6 (Pin_6), U401.8 (IO5)
- new net: J401.7 (Pin_7), U401.9 (IO6)
- new net: C301.2, R301.1
- new net: D402.2 (A), R404.2
- new net: Q301.3 (G), R303.1
- new net: R102.1, U101.9 (REF)
- new net: R307.1, U303.4 (EN)
- new net: C310.1, U303.1 (BST)
- new net: R308.1, R309.2, U303.3 (FB)
- new net: C310.2, L302.1, U303.6 (SW)
- new net: Q302.1 (D1/D2), Q302.8 (D1/D2)
- new net +3V3: C104.1, C105.1, C201.2, C202.2, C3012.2, C311.2, C313.2, C401.1, C402.1, J404.1 (Pin_1), J406.1 (Pin_1), J406.2 (Pin_2), J406.3 (Pin_3), J407.1 (Pin_1), J407.2 (Pin_2), J407.3 (Pin_3), L302.2, R308.2, R401.1, R402.1, R403.1, U101.12 (DCP), U101.13 (VCC), U201.16 (VCC), U201.4 (V3), U401.2 (3V3), U402.2 (Pin_2)
- new net BAT: BT1.1 (+), C304.2, C305.2, D301.1 (K), D303.2 (A), R304.2, U301.3 (BAT)
- new net BG: Q303.3 (G), R310.1, SW301.4 (A)
- new net BGND: C301.1, C302.1, C303.2, C304.1, C305.1, Q301.2 (S), Q302.6 (S2), Q302.7 (S2), Q303.1 (D), R306.2, U301.4 (GND)
- new net BT-: BT2.2 (-), C306.1, C307.1, Q302.2 (S1), Q302.3 (S1), U302.6 (VSS)
- new net ESP_EN: C403.2, J404.5 (Pin_5), R401.2, SW401.2, U401.41 (EN)
- new net ESP_IO0: J401.1 (Pin_1), J404.6 (Pin_6), R402.2, SW402.2, U401.3 (IO0)
- new net ESP_IO2: J401.3 (Pin_3), R404.1, U401.5 (IO2)
- new net ESP_RX: J404.3 (Pin_3), U201.2 (TXD), U401.38 (RXD0)
- new net ESP_SCL: J401.10 (Pin_10), U401.12 (IO9), U402.3 (Pin_3)
- new net ESP_SDA: J401.9 (Pin_9), U401.11 (IO8), U402.4 (Pin_4)
- new net ESP_TX: J404.2 (Pin_2), U201.3 (RXD), U401.37 (TXD0)
- new net U0_EN: Q202.3 (C)
- new net U0_IO0: Q201.3 (C)
- new net USB_1_D+: U101.8 (DP1), U201.5 (UD+)
- new net USB_1_D-: U101.7 (DM1), U201.6 (UD-)
- new net USB_2_D+: J403.4 (Pin_4), U101.6 (DP2), U401.20 (IO17)
- new net USB_2_D-: J403.3 (Pin_3), U101.5 (DM2), U401.19 (IO16)
- new net VCC: C308.2, C309.2, D302.1 (K), D303.1 (K), R307.2, R310.2, U303.5 (VIN)
- no-connect marks 7 -> 15
Other:
- note added: "1 不使用电池 2 使用电池供电"
- note added: "3.3V降压电路"
- note added: "USB"
- note added: "USB转串口"
- note added: "供电切换电路"
- note added: "充电电路"
- note added: "充电电路连接在一起再接系统地 充电电路接地时与4脚分开接地"
- note added: "电池和保护电路"
- moved on the sheet: USB101, USB102, USB103, USB104

Commit message: 更新电路图
Parts:
- removed H5, H6, H7, H8: MountingHole, MountingHole:MountingHole_2.2mm_M2_ISO14580, symbol Mechanical:MountingHole
- removed J406, J407: Conn_02x03_Counter_Clockwise, Connector_PinHeader_2.54mm:PinHeader_2x03_P2.54mm_Vertical, symbol Connector_Generic:Conn_02x03_Counter_Clockwise
- added C314: 22pF, Capacitor_SMD:C_0805_2012Metric, symbol Device:C_Small
- added J406, J407: Conn_02x03_Odd_Even, Connector_PinHeader_2.54mm:PinHeader_2x03_P2.54mm_Vertical, symbol Connector_Generic:Conn_02x03_Odd_Even
- renumbered C3012 to C312
Connections:
- net U0_EN is gone; now on net ESP_EN: Q202.3 (C)
- net U0_IO0 is gone; now on net ESP_IO0: Q201.3 (C)
- net +3V3: now also C313.1, C314.2, J406.1 (Pin_1), J406.3 (Pin_3), J406.5 (Pin_5), J407.1 (Pin_1), J407.3 (Pin_3), J407.5 (Pin_5); no longer C313.2, U101.13 (VCC)
- net +5V: now also C101.1, C102.1, U101.13 (VCC); no longer C101.2, C102.2
- net GND: now also C101.2, C102.2, C313.2, SW301.3 (C), SW301.6 (C), J406.2 (Pin_2), J406.4 (Pin_4), J406.6 (Pin_6), J407.2 (Pin_2), J407.4 (Pin_4), J407.6 (Pin_6); no longer C101.1, C102.1, C313.1, SW301.5 (B)
- net LR301: now reaches L301.1, R302.1, U301.8 (CSN)
- net LD301: now reaches D301.2 (A), L301.2, Q301.1 (D)
- net at SW301.1 (A): now also R310.1, SW301.4 (A)
- net at SW301.2 (B): now also Q303.3 (G), SW301.5 (B)
- net at R308.1, R309.2, U303.3 (FB): now also C314.1
- net LC301: now reaches C310.2, L302.1, U303.6 (SW)
- net DD301: now reaches Q302.1 (D1/D2), Q302.8 (D1/D2)
- removed net BG: Q303.3 (G), R310.1, SW301.4 (A)
Other:
- moved on the sheet: C101, C102, C313, R310, SW301

Commit message: 更新电路图
Connections:
- net +3V3: no longer C104.1, C105.1, U101.12 (DCP)
- net USB_2_D+: now also J403.7 (Pin_7), U401.23 (IO20); no longer J403.4 (Pin_4), U401.20 (IO17)
- net USB_2_D-: now also J403.6 (Pin_6), U401.22 (IO19); no longer J403.3 (Pin_3), U401.19 (IO16)
- net at U101.14 (V33): now also C104.1, C105.1, U101.12 (DCP)
- new net: J403.3 (Pin_3), U401.19 (IO16)
- new net: J403.4 (Pin_4), U401.20 (IO17)
- no-connect marks 15 -> 14
Changed lines of the file:
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@@
   (junction (at 265.43 87.63) (diameter 0) (color 0 0 0 0)
   )
-  (junction (at 101.6 48.26) (diameter 0) (color 0 0 0 0)
-  )
   (junction (at 143.51 224.79) (diameter 0) (color 0 0 0 0)
   )
@@
   (no_connect (at 46.99 109.22))
   (no_connect (at 172.72 57.15))
-  (no_connect (at 93.98 45.72))
   (no_connect (at 172.72 54.61))
   (wire (pts (xy 351.79 53.34) (xy 350.52 53.34))
@@
     (stroke (width 0) (type default) (color 0 0 0 0))
   )
-  (wire (pts (xy 101.6 50.8) (xy 101.6 48.26))
-    (stroke (width 0) (type default) (color 0 0 0 0))
-  )
   (polyline (pts (xy 323.85 19.05) (xy 323.85 62.23))
     (stroke (width 0) (type default) (color 0 0 0 0))
@@
     (stroke (width 0) (type default) (color 0 0 0 0))
   )
-  (wire (pts (xy 101.6 48.26) (xy 104.14 48.26))
-    (stroke (width 0) (type default) (color 0 0 0 0))
-  )
   (wire (pts (xy 93.98 124.46) (xy 93.98 125.73))
     (stroke (width 0) (type default) (color 0 0 0 0))
@@
     (stroke (width 0) (type default) (color 0 0 0 0))
   )
+  (wire (pts (xy 93.98 45.72) (xy 101.6 45.72))
+    (stroke (width 0) (type default) (color 0 0 0 0))
+  )
   (wire (pts (xy 88.9 27.94) (xy 88.9 26.67))
     (stroke (width 0) (type default) (color 0 0 0 0))
@@
     (stroke (width 0) (type default) (color 0 0 0 0))
   )
-  (wire (pts (xy 101.6 48.26) (xy 101.6 45.72))
+  (wire (pts (xy 101.6 45.72) (xy 101.6 50.8))
     (stroke (width 0) (type default) (color 0 0 0 0))
   )
@@
     (effects (font (size 1.27 1.27)) (justify right bottom))
   )
-  (label "USB_2_D-" (at 77.47 256.54 270)
+  (label "USB_2_D-" (at 85.09 256.54 270)
     (effects (font (size 1.27 1.27)) (justify right bottom))
   )
@@
     (effects (font (size 1.27 1.27)) (justify right bottom))
   )
-  (label "USB_2_D+" (at 80.01 256.54 270)
+  (label "USB_2_D+" (at 87.63 256.54 270)
     (effects (font (size 1.27 1.27)) (justify right bottom))
   )
@@
   (symbol (lib_id "power:+5V") (at 99.06 46.99 0) (unit 1)
     (in_bom yes) (on_board yes)
-    (property "Reference" "#PWR?" (id 0) (at 99.06 50.8 0)
+    (property "Reference" "#PWR0143" (id 0) (at 99.06 50.8 0)
       (effects (font (size 1.27 1.27)) hide)
     )
@@
     (pin "2")
   )
-  (symbol (lib_id "power:+3V3") (at 104.14 48.26 270) (unit 1)
-    (in_bom yes) (on_board yes) (fields_autoplaced)
-    (property "Reference" "#PWR0109" (id 0) (at 100.33 48.26 0)
-      (effects (font (size 1.27 1.27)) hide)
-    )
-    (property "Value" "+3V3" (id 1) (at 107.315 48.739 90)
-      (effects (font (size 1.27 1.27)) (justify left))
-    )
-    (property "Footprint" "" (id 2) (at 104.14 48.26 0)
-      (effects (font (size 1.27 1.27)) hide)
-    )
-    (property "Datasheet" "" (id 3) (at 104.14 48.26 0)
-      (effects (font (size 1.27 1.27)) hide)
-    )
-    (pin "1")
-  )
   (symbol (lib_id "Device:R_Small") (at 355.6 86.36 180) (unit 1)
     (in_bom yes) (on_board yes) (fields_autoplaced)
@@
       (reference "#PWR0108") (unit 1) (value "+5V") (footprint "")
     )
-    (path "/f4495dee-73d4-421c-a2ce-71eee75f8642"
-      (reference "#PWR0109") (unit 1) (value "+3V3") (footprint "")
-    )
     (path "/c2452d02-ff4b-4d74-b105-2198bcb8b0b3"
       (reference "#PWR0110") (unit 1) (value "GND") (footprint "")
@@
     )
     (path "/5e165934-7807-43ed-940e-6cc69877a643"
-      (reference "#PWR?") (unit 1) (value "+5V") (footprint "")
+      (reference "#PWR0143") (unit 1) (value "+5V") (footprint "")
     )
     (path "/0dad56a6-a4f8-4683-8fe9-d33a41651a89"
