File: Hardware/sbs3-board/sbs3-board.kicad_pcb (KiCad board)
At the start: 2 copper layers, 100 x 60 mm, 71 parts, among them J1 Conn_01x20_Male, J2 Conn_01x20_Male, J3 Conn_01x20_Male, J4 Conn_01x20_Male, J5 Conn_02x03_Odd_Even, J6 Conn_02x03_Odd_Even, Q1 PW2320, Q2 PW8205A8, Q3 SS8050, Q4 SS8050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

Commit message: 添加丝印
Routing:
- net /BT-: track 32.6 -> 35.9 mm
Other:
- board text added: "3V3 GND"
- board text added: "BOOT"
- board text added: "EN"
- board text added: "GND 1 2 TX RX 42 41 40 39 38 37 36 35 0 45 48 47 21 14 13"
- board text added: "GND 3V3 EN 4 5 6 7 15 16 17 18 8 19 20 3 46 9 10 11 12"
- board text added: "JLCJLCJLCJLC"
Changed lines of the file:
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@@
     (property "Sheetname" "")
     (attr smd)
-    (fp_text reference "C9" (at -2.7 0) (layer "F.SilkS")
+    (fp_text reference "C9" (at 2.6 0) (layer "F.SilkS")
       (effects (font (size 1 1) (thickness 0.15)))
     )
@@
     (property "Sheetname" "")
     (attr smd)
-    (fp_text reference "C3" (at -2.7 0.1) (layer "F.SilkS")
+    (fp_text reference "C3" (at 2.6 0) (layer "F.SilkS")
       (effects (font (size 1 1) (thickness 0.15)))
     )
@@
   (gr_arc locked (start 200 158.5) (mid 199.56066 159.56066) (end 198.5 160) (layer "Edge.Cuts") (width 0.2))
   (gr_line locked (start 200 158.5) (end 200 148.5) (layer "Edge.Cuts") (width 0.2))
+  (gr_text "JLCJLCJLCJLC" (at 185 131) (layer "F.SilkS")
+    (effects (font (size 1.5 1.2) (thickness 0.25)))
+  )
+  (gr_text "GND\n3V3\nEN\n4\n5\n6\n7\n15\n16\n17\n18\n8\n19\n20\n3\n46\n9\n10\n11\n12" (at 166 110 270) (layer "F.SilkS")
+    (effects (font (size 1.57 1) (thickness 0.15)) (justify left))
+  )
+  (gr_text "3V3 GND" (at 146.4 122.9) (layer "F.SilkS")
+    (effects (font (size 1 1) (thickness 0.15)))
+  )
+  (gr_text "EN" (at 174.1 152.1) (layer "F.SilkS")
+    (effects (font (size 1 1) (thickness 0.15)))
+  )
+  (gr_text "BOOT" (at 173.1 157.1) (layer "F.SilkS")
+    (effects (font (size 1 1) (thickness 0.15)))
+  )
+  (gr_text "GND\n1\n2\nTX\nRX\n42\n41\n40\n39\n38\n37\n36\n35\n0\n45\n48\n47\n21\n14\n13" (at 166 140 270) (layer "F.SilkS")
+    (effects (font (size 1.57 1) (thickness 0.15)) (justify right))
+  )
   (segment (start 190 152.9) (end 190 155.3) (width 0.25) (layer "F.Cu") (net 1))
   (segment (start 148.7875 134.2875) (end 147.54 133.04) (width 0.25) (layer "F.Cu") (net 1))
@@
   (via (at 172.8 153.7) (size 0.8) (drill 0.4) (layers "F.Cu" "B.Cu") (net 44))
   (via (at 166.9 153.4) (size 0.8) (drill 0.4) (layers "F.Cu" "B.Cu") (net 44))
+  (segment (start 166.9 154.7) (end 166.9 151.4) (width 1) (layer "B.Cu") (net 44))
   (segment (start 180 156) (end 173.1 156) (width 1) (layer "B.Cu") (net 44))
   (segment (start 166.9 154.7) (end 168.2 156) (width 1) (layer "B.Cu") (net 44))
@@
         (xy 122.9 123.9)
         (xy 122.9 121.9)
-        (xy 122.9 121.9)
         (xy 122.9 117.2)

Commit message: 添加sbs3开发板介绍和图片
Parts:
- moved C14 7.43 mm to (130.5, 124.0), turned to -90 degrees
- moved C13 7.16 mm to (128.5, 124.0), turned to -90 degrees
- moved R12 1.49 mm to (123.9, 106.0), turned to 90 degrees
- moved R11 1.41 mm to (126.0, 106.0), turned to -90 degrees
Routing:
- net Net-(Q4-Pad1): track 7.32 -> 2.20 mm
- net Net-(Q3-Pad1): track 8.44 -> 4.85 mm, vias 2 -> 0
- net +3V3: track 232.0 -> 235.3 mm
- net Net-(Q3-Pad2): track 9.81 -> 8.68 mm
- net GND: vias 68 -> 58
Other:
- board text added: "G 1 2 TX RX 42 41 40 39 38 37 36 35 0 45 48 47 21 14 13"
- board text added: "G V EN 4 5 6 7 15 16 17 18 8 19 20 3 46 9 10 11 12"
- board text removed: "GND 1 2 TX RX 42 41 40 39 38 37 36 35 0 45 48 47 21 14 13"
- board text removed: "GND 3V3 EN 4 5 6 7 15 16 17 18 8 19 20 3 46 9 10 11 12"
